File: Quad_Controller.sch (KiCad schematic (older format))
At the start: 40 parts, among them J1 Bat_Connect, J10 M1_Drive, J11 M2_Drive, J12 M3_Drive, J13 M4_Drive, J14 Conn_01x04_Female, J15 Conn_02x05_Odd_Even, J2 M1_VB, J3 M1_GND, J4 M2_VB, J5 M2_GND, J6 M3_VB, J7 M3_GND, J8 M4_VB, J9 M4_GND, SW1 SW_Push, U1 LM1117MPX-3_3_NOPB, U2 STM32F405RGT6, U3 LSM6DS3TR

Commit message: Major overhaul to fix schematic after transition to new library format
Parts:
- removed C3: 10uF, Capacitors_SMD:C_1206, symbol C
- removed U1: LM1117MPX-3_3_NOPB, digikey-footprints:SOT-223, symbol LM1117MPX-3_3_NOPB
- added C14: 470uF, Capacitor_SMD:C_1206_3216Metric, symbol Device:C
- added C3: 470pF, Capacitor_SMD:C_1206_3216Metric, symbol Device:C
- added D3: 1N5819, Diode_THT:D_DO-41_SOD81_P10.16mm_Horizontal, symbol Diode:1N5819
- added L1: 220uH, Inductor_SMD:L_Bourns_SRR1260, symbol Device:L
- added R10: 3.3k, Resistor_SMD:R_0603_1608Metric, symbol Device:R
- added R7: 0.33, Resistor_SMD:R_0805_2012Metric, symbol Device:R
- added R8: 2k, Resistor_SMD:R_0603_1608Metric, symbol Device:R
- added U1: MC34063AD, Package_SO:SOIC-8_3.9x4.9mm_P1.27mm, symbol Regulator_Switching:MC34063AD
- C1: value 10uF -> 100uF; footprint Capacitors_SMD:C_1206 -> Capacitor_SMD:C_1206_3216Metric; symbol C -> Device:C
- C10, C11, C12, C13, C2, C4, C5, C6, C7, C8, C9: footprint Capacitors_SMD:C_0603 -> Capacitors_SMD:C_0603_1608Metric; symbol C -> Device:C
- D1: footprint LEDs:LED_RGB_1210 -> LED_SMD:LED_RGB_1210; symbol LED_ARGB -> Device:LED_ARGB
- D2: footprint LEDs:LED_0603 -> LED_SMD:LED_0603_1608Metric; symbol LED -> Device:LED
- J1: footprint Connectors_Terminal_Blocks:TerminalBlock_bornier-2_P5.08mm -> TerminalBlock:TerminalBlock_bornier-2_P5.08mm; symbol Screw_Terminal_01x02 -> Connector:Screw_Terminal_01x02
- J10, J11, J12, J13: footprint Pin_Headers:Pin_Header_Straight_1x03_Pitch2.54mm -> Connector_Molex:Molex_PicoBlade_53047-0210_1x02_P1.25mm_Vertical; symbol Conn_01x03_Male -> Connector:Conn_01x02_Male
- J14: footprint Socket_Strips:Socket_Strip_Straight_1x04_Pitch2.54mm -> Connector_Molex:Molex_PicoBlade_53047-0410_1x04_P1.25mm_Vertical; symbol Conn_01x04_Female -> Connector:Conn_01x04_Female
- J15: footprint Pin_Headers:Pin_Header_Straight_2x05_Pitch1.27mm -> Tag-Connect:TC2030-NL_SMALL; symbol Conn_02x05_Odd_Even -> Tag-Connect:TC2030-CTX
- J2, J3, J4, J5, J6, J7, J8, J9: symbol Conn_01x01 -> Connector_Generic:Conn_01x01
- R1, R2, R4, R5, R6: footprint Resistors_SMD:R_0603 -> Resistors_SMD:R_0603_1608Metric; symbol R -> Device:R
- R3: footprint Resistors_SMD:R_0603 -> Resistor_SMD:R_0603_1608Metric; symbol R -> Device:R
- SW1: footprint Buttons_Switches_SMD:SW_SPST_B3U-1000P -> Button_Switch_SMD:SW_SPST_B3U-1000P; symbol SW_Push -> Switch:SW_Push
- U2: symbol STM32F405RGT6 -> dk_Embedded-Microcontrollers:STM32F405RGT6
- U3: symbol LSM6DS3TR -> dk_Motion-Sensors-IMUs-Inertial-Measurement-Units:LSM6DS3TR
Connections:
- net +12V: now also R7.2, U1.6 (Vin)
- net GND: no longer C10.2, C11.2, C12.2, C13.2, C2.1, C4.1, C5.1, C6.2, C7.2, C8.2, C9.2, J10.1 (Pin_1), J11.1 (Pin_1), J12.1 (Pin_1), J13.1 (Pin_1), J14.2 (Pin_2), J15.5 (Pin_5), J15.6 (Pin_6), R6.2, SW1.2, U2.12 (VSSA), U2.18 (VSS), U2.63 (VSS), U3.6 (GND), U3.7 (GND)
- net M1S: now also J10.2 (Pin_2); no longer J10.3 (Pin_3)
- net M2S: now also J11.2 (Pin_2); no longer J11.3 (Pin_3)
- net M3S: now also J12.2 (Pin_2); no longer J12.3 (Pin_3)
- net M4S: now also J13.2 (Pin_2); no longer J13.3 (Pin_3)
- net RST: now also J15.3 (~RESET~), SW1.2; no longer J15.1 (Pin_1), SW1.1
- net SPI_MISO: now also U3.2 (SDx); no longer U3.1 (SDO/SA0)
- net SPI_MOSI: now also U3.3 (SCx); no longer U3.14 (SDA)
- net SWCLK: now also J15.4 (SWCLK/TCK); no longer J15.2 (Pin_2)
- net SWDIO: now also J15.2 (SWDIO/TMS); no longer J15.4 (Pin_4)
- net SWIM: now also J15.6 (SWO/TDO); no longer J15.3 (Pin_3)
- net VDD: now also C13.2, J15.1 (VCC), C14.2, L1.2, R10.1; no longer C13.1, J15.7 (Pin_7), J15.8 (Pin_8)
- new net: R7.1, U1.1 (SwC), U1.7 (Ipk), U1.8 (DC)
- new net: D3.1 (K), L1.1, U1.2 (SwE)
- new net: C3.1, U1.3 (TC)
- new net: R10.2, R8.1, U1.5 (Vfb)
- new net GNDD: C10.2, C11.2, C12.2, C13.1, C14.1, C2.1, C3.2, C4.1, C5.1, C6.2, C7.2, C8.2, C9.2, D3.2 (A), J10.1 (Pin_1), J11.1 (Pin_1), J12.1 (Pin_1), J13.1 (Pin_1), J14.2 (Pin_2), J15.5 (GND), R6.2, R8.2, SW1.1, U1.4 (GND), U2.12 (VSSA), U2.18 (VSS), U2.63 (VSS), U3.6 (GND), U3.7 (GND)
Other:
- note added: "3.3V Switching Regulator"
- note added: "Microcontroller"
- note added: "Motor Connections"
- note added: "out = R2/R1=3.3/2=3.3125V"
- note removed: "3.3V Regulator"
- note removed: "Micro"
- moved on the sheet: C1, C10, C11, C13, C2, C4, C5, C6, C7, C8, C9, D1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

Commit message: Fixing dumb mistake Capacitors -> Capacitor (same with resistor)
Parts:
- C10, C11, C12, C13, C2, C4, C5, C6, C7, C8, C9: footprint Capacitors_SMD:C_0603_1608Metric -> Capacitor_SMD:C_0603_1608Metric
- L1: footprint Inductor_SMD:L_Bourns_SRR1260 -> Inductor_SMD:L_Bourns_SRN6045TA
- R1, R2, R4, R5, R6: footprint Resistors_SMD:R_0603_1608Metric -> Resistor_SMD:R_0603_1608Metric
Changed lines of the file:
@@
 F 0 "C5" H 3525 5200 50  0000 L CNN
 F 1 "2.2uF" H 3525 5000 50  0000 L CNN
-F 2 "Capacitors_SMD:C_0603_1608Metric" H 3538 4950 50  0001 C CNN
+F 2 "Capacitor_SMD:C_0603_1608Metric" H 3538 4950 50  0001 C CNN
 F 3 "" H 3500 5100 50  0001 C CNN
 	1    3500 5100
@@
 F 0 "C11" H 7125 6450 50  0000 L CNN
 F 1 "100nF" H 7125 6250 50  0000 L CNN
-F 2 "Capacitors_SMD:C_0603_1608Metric" H 7138 6200 50  0001 C CNN
+F 2 "Capacitor_SMD:C_0603_1608Metric" H 7138 6200 50  0001 C CNN
 F 3 "" H 7100 6350 50  0001 C CNN
 	1    7100 6350
@@
 F 0 "C10" H 7475 6350 50  0000 L CNN
 F 1 "100nF" H 7475 6150 50  0000 L CNN
-F 2 "Capacitors_SMD:C_0603_1608Metric" H 7488 6100 50  0001 C CNN
+F 2 "Capacitor_SMD:C_0603_1608Metric" H 7488 6100 50  0001 C CNN
 F 3 "" H 7450 6250 50  0001 C CNN
 	1    7450 6250
@@
 F 0 "C9" H 7125 6250 50  0000 L CNN
 F 1 "100nF" H 7125 6050 50  0000 L CNN
-F 2 "Capacitors_SMD:C_0603_1608Metric" H 7138 6000 50  0001 C CNN
+F 2 "Capacitor_SMD:C_0603_1608Metric" H 7138 6000 50  0001 C CNN
 F 3 "" H 7100 6150 50  0001 C CNN
 	1    7100 6150
@@
 F 0 "C8" H 7475 6150 50  0000 L CNN
 F 1 "100nF" H 7475 5950 50  0000 L CNN
-F 2 "Capacitors_SMD:C_0603_1608Metric" H 7488 5900 50  0001 C CNN
+F 2 "Capacitor_SMD:C_0603_1608Metric" H 7488 5900 50  0001 C CNN
 F 3 "" H 7450 6050 50  0001 C CNN
 	1    7450 6050
@@
 F 0 "C7" H 7125 6050 50  0000 L CNN
 F 1 "100nF" H 7125 5850 50  0000 L CNN
-F 2 "Capacitors_SMD:C_0603_1608Metric" H 7138 5800 50  0001 C CNN
+F 2 "Capacitor_SMD:C_0603_1608Metric" H 7138 5800 50  0001 C CNN
 F 3 "" H 7100 5950 50  0001 C CNN
 	1    7100 5950
@@
 F 0 "C6" H 7275 5700 50  0000 L CNN
 F 1 "4.7uF" H 7275 5500 50  0000 L CNN
-F 2 "Capacitors_SMD:C_0603_1608Metric" H 7288 5450 50  0001 C CNN
+F 2 "Capacitor_SMD:C_0603_1608Metric" H 7288 5450 50  0001 C CNN
 F 3 "" H 7250 5600 50  0001 C CNN
 	1    7250 5600
@@
 F 0 "C12" H 8125 1350 50  0000 L CNN
 F 1 "100nF" H 8125 1150 50  0000 L CNN
-F 2 "Capacitors_SMD:C_0603_1608Metric" H 8138 1100 50  0001 C CNN
+F 2 "Capacitor_SMD:C_0603_1608Metric" H 8138 1100 50  0001 C CNN
 F 3 "" H 8100 1250 50  0001 C CNN
 	1    8100 1250
@@
 F 0 "C13" H 7175 2100 50  0000 L CNN
 F 1 "100nF" H 7175 1900 50  0000 L CNN
-F 2 "Capacitors_SMD:C_0603_1608Metric" H 7188 1850 50  0001 C CNN
+F 2 "Capacitor_SMD:C_0603_1608Metric" H 7188 1850 50  0001 C CNN
 F 3 "" H 7150 2000 50  0001 C CNN
 	1    7150 2000
@@
 F 0 "R1" V 2080 1900 50  0000 C CNN
 F 1 "56k" V 2000 1900 50  0000 C CNN
-F 2 "Resistors_SMD:R_0603_1608Metric" V 1930 1900 50  0001 C CNN
+F 2 "Resistor_SMD:R_0603_1608Metric" V 1930 1900 50  0001 C CNN
 F 3 "" H 2000 1900 50  0001 C CNN
 	1    2000 1900
@@
 F 0 "R2" V 2080 2300 50  0000 C CNN
 F 1 "20k" V 2000 2300 50  0000 C CNN
-F 2 "Resistors_SMD:R_0603_1608Metric" V 1930 2300 50  0001 C CNN
+F 2 "Resistor_SMD:R_0603_1608Metric" V 1930 2300 50  0001 C CNN
 F 3 "" H 2000 2300 50  0001 C CNN
 	1    2000 2300
@@
 F 0 "C2" H 10325 2650 50  0000 L CNN
 F 1 "100nF" H 10325 2450 50  0000 L CNN
-F 2 "Capacitors_SMD:C_0603_1608Metric" H 10338 2400 50  0001 C CNN
+F 2 "Capacitor_SMD:C_0603_1608Metric" H 10338 2400 50  0001 C CNN
 F 3 "" H 10300 2550 50  0001 C CNN
 	1    10300 2550
@@
 F 0 "C4" H 3525 5000 50  0000 L CNN
 F 1 "2.2uF" H 3525 4800 50  0000 L CNN
-F 2 "Capacitors_SMD:C_0603_1608Metric" H 3538 4750 50  0001 C CNN
+F 2 "Capacitor_SMD:C_0603_1608Metric" H 3538 4750 50  0001 C CNN
 F 3 "" H 3500 4900 50  0001 C CNN
 	1    3500 4900
@@
 F 0 "R4" V 7880 3500 50  0000 C CNN
 F 1 "1k" V 7800 3500 50  0000 C CNN
-F 2 "Resistors_SMD:R_0603_1608Metric" V 7730 3500 50  0001 C CNN
+F 2 "Resistor_SMD:R_0603_1608Metric" V 7730 3500 50  0001 C CNN
 F 3 "" H 7800 3500 50  0001 C CNN
 	1    7800 3500
@@
 F 0 "R5" V 7880 3700 50  0000 C CNN
 F 1 "1k" V 7800 3700 50  0000 C CNN
-F 2 "Resistors_SMD:R_0603_1608Metric" V 7730 3700 50  0001 C CNN
+F 2 "Resistor_SMD:R_0603_1608Metric" V 7730 3700 50  0001 C CNN
 F 3 "" H 7800 3700 50  0001 C CNN
 	1    7800 3700
@@
 F 0 "R6" V 7730 4500 50  0000 C CNN
 F 1 "1k" V 7650 4500 50  0000 C CNN
-F 2 "Resistors_SMD:R_0603_1608Metric" V 7580 4500 50  0001 C CNN
+F 2 "Resistor_SMD:R_0603_1608Metric" V 7580 4500 50  0001 C CNN
 F 3 "" H 7650 4500 50  0001 C CNN
 	1    7650 4500
@@
 F 0 "L1" V 5600 2500 50  0000 C CNN
 F 1 "220uH" V 5450 2500 50  0000 C CNN
-F 2 "Inductor_SMD:L_Bourns_SRR1260" H 5500 2500 50  0001 C CNN
+F 2 "Inductor_SMD:L_Bourns_SRN6045TA" H 5500 2500 50  0001 C CNN
 F 3 "~" H 5500 2500 50  0001 C CNN
 	1    5500 2500
@@
 	6150 2800 5800 2800
 $Comp
-L power:GND #PWR?
+L power:GND #PWR0103
 U 1 1 5D295A5F
 P 3250 1850
-F 0 "#PWR?" H 3250 1600 50  0001 C CNN
+F 0 "#PWR0103" H 3250 1600 50  0001 C CNN
 F 1 "GND" H 3250 1700 50  0000 C CNN
 F 2 "" H 3250 1850 50  0001 C CNN
@@
 $EndComp
 $Comp
-L power:VDD #PWR?
+L power:VDD #PWR0106
 U 1 1 5D295C09
 P 10100 4050
-F 0 "#PWR?" H 10100 3900 50  0001 C CNN
+F 0 "#PWR0106" H 10100 3900 50  0001 C CNN
 F 1 "VDD" H 10100 4200 50  0000 C CNN
 F 2 "" H 10100 4050 50  0001 C CNN

Commit message: Adding some small updates (redoing layout with components on back of board)
Parts:
- C1: footprint Capacitor_SMD:C_1206_3216Metric -> Capacitor_SMD:CP_Elec_5x5.3
- C14, C3: footprint Capacitor_SMD:C_1206_3216Metric -> Capacitor_SMD:C_0603_1608Metric
Connections:
- net M1S: now also U2.16 (PA2); no longer U2.62 (PB9)
- net M2S: now also U2.33 (PB12); no longer U2.51 (PC10)
- net M3S: now also U2.51 (PC10); no longer U2.33 (PB12)
- net M4S: now also U2.62 (PB9); no longer U2.16 (PA2)
- net SPI_MISO: now also U3.1 (SDO/SA0); no longer U3.2 (SDx)
- net SPI_MOSI: now also U3.14 (SDA); no longer U3.3 (SCx)
Changed lines of the file:
@@
 Wire Wire Line
 	8000 2400 8000 2500
-Text Label 8700 1650 0    60   ~ 0
+Text Label 8700 1550 0    60   ~ 0
 SPI_MISO
 Wire Wire Line
-	8700 1650 8450 1650
+	8700 1550 8450 1550
 $Comp
 L Connector_Generic:Conn_01x01 J2
@@
 F 0 "C1" V 3750 1800 50  0000 L CNN
 F 1 "100uF" V 3450 1750 50  0000 L CNN
-F 2 "Capacitor_SMD:C_1206_3216Metric" H 3638 1700 50  0001 C CNN
+F 2 "Capacitor_SMD:CP_Elec_5x5.3" H 3638 1700 50  0001 C CNN
 F 3 "http://datasheets.avx.com/TAJ.pdf" H 3600 1850 50  0001 C CNN
 	1    3600 1850
@@
 Wire Wire Line
 	5850 7050 5850 6650
-Text Label 8700 1750 0    60   ~ 0
+Text Label 8700 2050 0    60   ~ 0
 SPI_MOSI
 Wire Wire Line
-	8700 1750 8450 1750
+	8700 2050 8450 2050
 Text Label 4650 5000 1    60   ~ 0
 SPI_MISO
@@
 	4850 5000 4850 5450
 Text Label 6250 7050 3    60   ~ 0
-M3S
+M2S
 Wire Wire Line
 	6250 7050 6250 6650
 Text Label 5050 5000 1    60   ~ 0
-M4S
+M1S
 Wire Wire Line
 	5050 5000 5050 5450
 Text Label 4650 7050 3    60   ~ 0
-M2S
+M3S
 Text Label 3550 7050 3    60   ~ 0
-M1S
+M4S
 Wire Wire Line
 	4650 7050 4650 6650
@@
 F 0 "C3" V 4000 2450 50  0000 L CNN
 F 1 "470pF" V 3700 2400 50  0000 L CNN
-F 2 "Capacitor_SMD:C_1206_3216Metric" H 3888 2350 50  0001 C CNN
+F 2 "Capacitor_SMD:C_0603_1608Metric" H 3888 2350 50  0001 C CNN
 F 3 "http://datasheets.avx.com/TAJ.pdf" H 3850 2500 50  0001 C CNN
 	1    3850 2500
@@
 F 0 "C14" H 5825 3150 50  0000 L CNN
 F 1 "470uF" H 5825 2950 50  0000 L CNN
-F 2 "Capacitor_SMD:C_1206_3216Metric" H 5838 2900 50  0001 C CNN
+F 2 "Capacitor_SMD:C_0603_1608Metric" H 5838 2900 50  0001 C CNN
 F 3 "http://datasheets.avx.com/TAJ.pdf" H 5800 3050 50  0001 C CNN
 	1    5800 3050

Commit message: Connecting missed pad and clarifying formula for output of switching regulator)
Other:
- note added: "FR1"
- note added: "FR2"
- note added: "out=1.25*(1+FR2/FR1)=3.3125V"
- note removed: "out = R2/R1=3.3/2=3.3125V"
Changed lines of the file:
@@
 EESchema Schematic File Version 4
 LIBS:Quad_Controller-cache
-EELAYER 26 0
+EELAYER 29 0
 EELAYER END
 $Descr A4 11693 8268
@@
 Motor Connections
 Text Notes 5900 2700 0    50   ~ 0
-out = R2/R1=3.3/2=3.3125V
+out=1.25*(1+FR2/FR1)=3.3125V
 Wire Wire Line
 	4750 1950 5300 1950
@@
 	-1   0    0    1
 $EndComp
+Text Notes 4850 3100 0    50   ~ 0
+FR1
+Text Notes 5000 2950 0    50   ~ 0
+FR2
 $EndSCHEMATC
